File: kicad/cpu.kicad_sch (KiCad schematic)
At the start: 7 parts, among them U3 W65C02SxP

Commit message: minor schematic updayes
Parts:
- added R42: R, Resistor_THT:R_Axial_DIN0207_L6.3mm_D2.5mm_P10.16mm_Horizontal, symbol Device:R
Connections:
- net RDY: now also R42.2
- net VCC: now also R42.1
Other:
- moved on the sheet: R19, R20, R21, R22, R23

Commit message: value updates, fix ROM ~WE
Parts:
- R19, R20, R21, R22, R23: value R -> 4K7
Other:
- moved on the sheet: R20
Changed lines of the file:
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@@
 	(wire
 		(pts
-			(xy 257.81 62.23) (xy 261.62 62.23)
+			(xy 259.08 60.96) (xy 262.89 60.96)
 		)
 		(stroke
@@
 	(wire
 		(pts
-			(xy 261.62 62.23) (xy 261.62 59.69)
+			(xy 262.89 60.96) (xy 262.89 58.42)
 		)
 		(stroke
@@
 	(hierarchical_label "~{SO}"
 		(shape bidirectional)
-		(at 257.81 62.23 180)
+		(at 259.08 60.96 180)
 		(effects
 			(font
@@
 			)
 		)
-		(property "Value" "R"
+		(property "Value" "4K7"
 			(at 210.82 55.8799 0)
 			(effects
@@
 			)
 		)
-		(property "Value" "R"
+		(property "Value" "4K7"
 			(at 229.87 55.8799 0)
 			(effects
@@
 	(symbol
 		(lib_id "power:VCC")
-		(at 261.62 52.07 0)
+		(at 262.89 50.8 0)
 		(unit 1)
 		(exclude_from_sim no)
@@
 		(fields_autoplaced yes)
 		(property "Reference" "#PWR035"
-			(at 261.62 55.88 0)
+			(at 262.89 54.61 0)
 			(effects
 				(font
@@
 		)
 		(property "Value" "VCC"
-			(at 261.62 46.99 0)
+			(at 262.89 45.72 0)
 			(effects
 				(font
@@
 		)
 		(property "Footprint" ""
-			(at 261.62 52.07 0)
+			(at 262.89 50.8 0)
 			(effects
 				(font
@@
 		)
 		(property "Datasheet" ""
-			(at 261.62 52.07 0)
+			(at 262.89 50.8 0)
 			(effects
 				(font
@@
 		)
 		(property "Description" "Power symbol creates a global label with name \"VCC\""
-			(at 261.62 52.07 0)
+			(at 262.89 50.8 0)
 			(effects
 				(font
@@
 			)
 		)
-		(property "Value" "R"
+		(property "Value" "4K7"
 			(at 246.38 55.8799 0)
 			(effects
@@
 			)
 		)
-		(property "Value" "R"
+		(property "Value" "4K7"
 			(at 193.04 55.8799 0)
 			(effects
@@
 	(symbol
 		(lib_id "Device:R")
-		(at 261.62 55.88 0)
+		(at 262.89 54.61 0)
 		(unit 1)
 		(exclude_from_sim no)
@@
 		(fields_autoplaced yes)
 		(property "Reference" "R20"
-			(at 264.16 54.6099 0)
+			(at 265.43 53.3399 0)
 			(effects
 				(font
@@
 			)
 		)
-		(property "Value" "R"
-			(at 264.16 57.1499 0)
+		(property "Value" "4K7"
+			(at 265.43 55.8799 0)
 			(effects
 				(font
@@
 		)
 		(property "Footprint" "Resistor_THT:R_Axial_DIN0207_L6.3mm_D2.5mm_P10.16mm_Horizontal"
-			(at 259.842 55.88 90)
+			(at 261.112 54.61 90)
 			(effects
 				(font
@@
 		)
 		(property "Datasheet" "~"
-			(at 261.62 55.88 0)
+			(at 262.89 54.61 0)
 			(effects
 				(font
@@
 		)
 		(property "Description" "Resistor"
-			(at 261.62 55.88 0)
-			(effects
-				(font
+			(at 262.89 54.61 0)
+			(effects
+				(font
